Commit message: Faze4Gui

File: faze4_description/urdf/faze4_description.urdf.xacro (robot description, xacro)
@@ -200,5 +200,5 @@
     <origin
       xyz="0.32 0 0"
-      rpy="3.1416 -6.3895E-16 -3.3" />
+      rpy="3.1416 0 -3.3" />
     <parent
       link="${prefix}link2" />
@@ -207,5 +207,5 @@
     <axis
       xyz="0 0 -1" />
-    <limit lower="-0.3" upper="2.35" effort="1000.0" velocity="0.3"/>
+    <limit lower="-0.3" upper="2.61799" effort="1000.0" velocity="0.3"/>
   </joint>
   <link
@@ -254,5 +254,5 @@
     <origin
       xyz="0 -0.0735 0"
-      rpy="-0.5648 -0.78173 1.7809" />
+      rpy="-0.5648 -0.675 1.7809" />
     <parent
       link="${prefix}link3" />
@@ -308,5 +308,5 @@
     <origin
       xyz="0.037114 0.22683 0.10011"
-      rpy="2.2965 -0.74045 -0.57161" />
+      rpy="2.16 -0.74045 -0.57161" />
     <parent
       link="${prefix}link4" />
@@ -336,5 +336,5 @@
       <origin
         xyz="0 0 0"
-        rpy="0 0 0" />
+        rpy="0 0 0.77" />
       <geometry>
         <mesh
@@ -350,5 +350,5 @@
       <origin
         xyz="0 0 0"
-        rpy="0 0 0" />
+        rpy="0 0 0.77" />
       <geometry>
         <mesh
@@ -362,5 +362,5 @@
     <origin
       xyz="0 0 -0.042312"
-      rpy="-3.1416 2.5362E-15 0.2419" />
+      rpy="-3.1416 0 0" />
     <parent
       link="${prefix}link5" />
@@ -369,4 +369,55 @@
     <axis
       xyz="0 0 1" />
+  </joint>
+  <link
+    name="${prefix}link7">
+    <inertial>
+      <origin
+        xyz="0 0 0"
+        rpy="0 0 0" />
+      <mass
+        value="0.011" />
+      <inertia
+        ixx="1.5488534576213277e-05"
+        ixy="0"
+        ixz="0"
+        iyy="1.5488915081958018e-05"
+        iyz="0"
+        izz="4.689528721728688e-07" />
+    </inertial>
+    <visual>
+      <origin
+        xyz="0 0 0"
+        rpy="0 0 0" />
+      <geometry>
+        <mesh
+          filename="package://faze4_description/meshes/marker.stl" />
+      </geometry>
+      <material
+        name="">
+        <color
+          rgba="0.792156862745098 0.819607843137255 0.933333333333333 1" />
+      </material>
+    </visual>
+    <collision>
+      <origin
+        xyz="0 0 0"
+        rpy="0 0 0" />
+      <geometry>
+        <mesh
+          filename="package://faze4_description/meshes/marker.stl" />
+      </geometry>
+    </collision>
+  </link>
+  <joint
+    name="${prefix}joint7"
+    type="fixed">
+    <origin
+      xyz="0 0.1 0.024"
+      rpy="1.57 0 0" />
+    <parent
+      link="${prefix}link6" />
+    <child
+      link="${prefix}link7" />
   </joint>
 </xacro:macro>

File: faze4_moveit_config/config/faze4_arm.xacro (robot description, xacro)
@@ -8,8 +8,9 @@
     <!--SUBGROUPS - Groups can also be formed by referencing to already defined group names-->
     <group name="faze4_arm">
-      <chain base_link="faze4_base_link" tip_link="faze4_link6" />
+      <chain base_link="faze4_base_link" tip_link="faze4_link7" />
     </group>
     <group name="gripper">
         <link name="faze4_link6" />
+        <link name="faze4_link7" />
     </group>
     <!--GROUP STATES - Purpose - Define a named state for a particular group, in terms of joint values. This is useful to define states like 'folded arms'-->
@@ -39,5 +40,5 @@
     </group_state>
     <!--END EFFECTOR - Purpose - Represent information about an end effector.-->
-    <end_effector name="gripper" parent_link="faze4_link6" group="gripper" parent_group="faze4_arm"/>
+    <end_effector name="gripper" parent_link="faze4_link7" group="gripper" />
     <!--VIRTUAL JOINT - Purpose - this element defines a virtual joint between a robot link and an external frame of reference (considered fixed with respect to the robot)-->
     <virtual_joint name="virtual_joint" type="fixed" parent_frame="world" child_link="world" />
